File: nrf5340_power.sch (KiCad schematic (older format))
At the start: 9 parts

Commit message: update
Parts:
- removed U?: AP2112K-3.3, Package_TO_SOT_SMD:SOT-23-5, symbol Regulator_Linear:AP2112K-3.3
- added U2: AP2112K-3.3, Package_TO_SOT_SMD:SOT-23-5, symbol Regulator_Linear:AP2112K-3.3
- gave numbers to parts that had none: 8
Connections:
- net GND: now also U2.2 (GND)
- net VDD_nRF: now also U2.5 (VOUT)
- net at C29.1, D2.1 (K), Q1.2 (S)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: now also U2.1 (VIN)
- net at R6.2: now also U2.3 (EN)
Other:
- note added: "VERY bright, might choose a bigger res"
Changed lines of the file:
@@
 EESchema Schematic File Version 4
-LIBS:nrf5340_module-cache
 EELAYER 30 0
 EELAYER END
 $Descr A4 11693 8268
 encoding utf-8
-Sheet 3 7
+Sheet 3 3
 Title ""
 Date ""
-Rev ""
+Rev "1.0"
 Comp ""
 Comment1 ""
@@
 $EndDescr
 $Comp
-L Device:Q_PMOS_GSD Q?
+L Device:Q_PMOS_GSD Q1
 U 1 1 5E164004
 P 1450 1050
-F 0 "Q?" H 1655 1096 50  0000 L CNN
+F 0 "Q1" H 1655 1096 50  0000 L CNN
 F 1 "Q_PMOS_GSD" H 1655 1005 50  0000 L CNN
 F 2 "Package_TO_SOT_SMD:SOT-23" H 1650 1150 50  0001 C CNN
@@
 $EndComp
 $Comp
-L Device:R_Small R?
+L Device:R_Small R4
 U 1 1 5E1648ED
 P 1000 1550
-F 0 "R?" H 750 1600 50  0000 L CNN
+F 0 "R4" H 750 1600 50  0000 L CNN
 F 1 "100k" H 750 1500 50  0000 L CNN
 F 2 "Resistor_SMD:R_0201_0603Metric" H 1000 1550 50  0001 C CNN
@@
 $EndComp
 $Comp
-L Device:D_Zener_Small D?
+L Device:D_Zener_Small D2
 U 1 1 5E165282
 P 1300 1400
-F 0 "D?" H 1300 1195 50  0000 C CNN
+F 0 "D2" H 1300 1195 50  0000 C CNN
 F 1 "MBR120" H 1300 1286 50  0000 C CNN
 F 2 "Diode_SMD:D_SOD-123" V 1300 1400 50  0001 C CNN
@@
 $EndComp
 $Comp
-L Device:C_Small C?
+L Device:C_Small C29
 U 1 1 5E165C53
 P 1550 1550
-F 0 "C?" H 1642 1596 50  0000 L CNN
+F 0 "C29" H 1642 1596 50  0000 L CNN
 F 1 "10uF" H 1642 1505 50  0000 L CNN
 F 2 "Capacitor_SMD:C_0201_0603Metric" H 1550 1550 50  0001 C CNN
@@
 $EndComp
 $Comp
-L Device:C_Small C?
+L Device:C_Small C30
 U 1 1 5E16615D
 P 2800 1550
-F 0 "C?" H 2892 1596 50  0000 L CNN
+F 0 "C30" H 2892 1596 50  0000 L CNN
 F 1 "10uF" H 2892 1505 50  0000 L CNN
 F 2 "Capacitor_SMD:C_0201_0603Metric" H 2800 1550 50  0001 C CNN
@@
 $EndComp
 $Comp
-L Device:R_Small R?
+L Device:R_Small R6
 U 1 1 5E1662E7
 P 2000 1500
-F 0 "R?" V 2100 1500 50  0000 C CNN
+F 0 "R6" V 2100 1500 50  0000 C CNN
 F 1 "100k" V 2200 1500 50  0000 C CNN
 F 2 "Resistor_SMD:R_0201_0603Metric" H 2000 1500 50  0001 C CNN
@@
 	1    2000 1500
 	0    -1   1    0
-$EndComp
-$Comp
-L Regulator_Linear:AP2112K-3.3 U?
-U 1 1 5E166BA6
-P 2450 1500
-F 0 "U?" H 2450 1842 50  0000 C CNN
-F 1 "AP2112K-3.3" H 2450 1751 50  0000 C CNN
-F 2 "Package_TO_SOT_SMD:SOT-23-5" H 2450 1825 50  0001 C CNN
-F 3 "https://www.diodes.com/assets/Datasheets/AP2112.pdf" H 2450 1600 50  0001 C CNN
-	1    2450 1500
-	1    0    0    -1
 $EndComp
 Text GLabel 2850 1400 2    50   Input ~ 0
@@
 Connection ~ 1850 1400
 $Comp
-L power:GND #PWR?
+L power:GND #PWR018
 U 1 1 5E177C45
 P 2800 1700
-F 0 "#PWR?" H 2800 1450 50  0001 C CNN
+F 0 "#PWR018" H 2800 1450 50  0001 C CNN
 F 1 "GND" H 2805 1527 50  0000 C CNN
 F 2 "" H 2800 1700 50  0001 C CNN
@@
 $EndComp
 $Comp
-L power:GND #PWR?
+L power:GND #PWR017
 U 1 1 5E177E44
 P 2450 1850
-F 0 "#PWR?" H 2450 1600 50  0001 C CNN
+F 0 "#PWR017" H 2450 1600 50  0001 C CNN
 F 1 "GND" H 2455 1677 50  0000 C CNN
 F 2 "" H 2450 1850 50  0001 C CNN
@@
 $EndComp
 $Comp
-L power:GND #PWR?
+L power:GND #PWR016
 U 1 1 5E17842E
 P 1550 1700
-F 0 "#PWR?" H 1550 1450 50  0001 C CNN
+F 0 "#PWR016" H 1550 1450 50  0001 C CNN
 F 1 "GND" H 1555 1527 50  0000 C CNN
 F 2 "" H 1550 1700 50  0001 C CNN
@@
 $EndComp
 $Comp
-L power:GND #PWR?
+L power:GND #PWR014
 U 1 1 5E178752
 P 1000 1700
-F 0 "#PWR?" H 1000 1450 50  0001 C CNN
+F 0 "#PWR014" H 1000 1450 50  0001 C CNN
 F 1 "GND" H 1005 1527 50  0000 C CNN
 F 2 "" H 1000 1700 50  0001 C CNN
@@
 	2800 1400 2750 1400
 $Comp
-L Device:LED D?
+L Device:LED D1
 U 1 1 5E1852C7
 P 1000 2850
-F 0 "D?" V 1039 2733 50  0000 R CNN
+F 0 "D1" V 1039 2733 50  0000 R CNN
 F 1 "LED" V 948 2733 50  0000 R CNN
 F 2 "LED_SMD:LED_0402_1005Metric" H 1000 2850 50  0001 C CNN
@@
 VDD_nRF
 $Comp
-L Device:R_Small R?
+L Device:R_Small R5
 U 1 1 5E18637C
 P 1000 2550
-F 0 "R?" H 850 2600 50  0000 L CNN
+F 0 "R5" H 850 2600 50  0000 L CNN
 F 1 "68R" H 800 2500 50  0000 L CNN
 F 2 "Resistor_SMD:R_0201_0603Metric" H 1000 2550 50  0001 C CNN
@@
 	1000 3000 1000 3050
 $Comp
-L power:GND #PWR?
+L power:GND #PWR015
 U 1 1 5E187B31
 P 1000 3050
-F 0 "#PWR?" H 1000 2800 50  0001 C CNN
+F 0 "#PWR015" H 1000 2800 50  0001 C CNN
 F 1 "GND" H 1005 2877 50  0000 C CNN
 F 2 "" H 1000 3050 50  0001 C CNN
@@
 	1    0    0    -1
 $EndComp
+$Comp
+L Regulator_Linear:AP2112K-3.3 U2
+U 1 1 602514BE
+P 2450 1500
+F 0 "U2" H 2450 1842 50  0000 C CNN
+F 1 "AP2112K-3.3" H 2450 1751 50  0000 C CNN
+F 2 "Package_TO_SOT_SMD:SOT-23-5" H 2450 1825 50  0001 C CNN
+F 3 "https://www.diodes.com/assets/Datasheets/AP2112.pdf" H 2450 1600 50  0001 C CNN
+	1    2450 1500
+	1    0    0    -1
+$EndComp
+Text Notes 1100 2600 0    50   ~ 0
+VERY bright, might choose a bigger res
 $EndSCHEMATC
